Commit message: Add base_link

File: my_rb1_description/urdf/my_rb1_robot.urdf (robot description, URDF)
Before this commit: robot rb1_robot, 7 links, 6 joints
Links:
- removed link back_caster
- removed link base_footprint
- removed link front_caster
- removed link front_laser
- removed link left_wheel
- removed link right_wheel
- link base_link: mass None -> 18; geometry collision cylinder length=0.30 radius=0.25; visual cylinder length=0.30 radius=0.25
Joints:
- removed joint base_link_back_caster_joint
- removed joint base_link_front_caster_joint
- removed joint base_link_front_laser_joint
- removed joint base_link_left_wheel_joint
- removed joint base_link_plate_joint
- removed joint base_link_right_wheel_joint

Commit message: Add both caster wheels and both drive wheels

File: my_rb1_description/urdf/my_rb1_robot.urdf (robot description, URDF)
Before this commit: robot rb1_robot, 1 links, 0 joints
Links:
- added link back_caster, mass 1; collision sphere radius=0.025; collision sphere radius=0.03
- added link base_footprint
- added link front_caster, mass 1; collision sphere radius=0.025; collision sphere radius=0.03
- added link link_left_wheel, mass 1; collision cylinder length=0.04 radius=0.025; collision cylinder length=0.06 radius=0.01
- added link link_right_wheel, mass 1; collision cylinder length=0.04 radius=0.025; collision cylinder length=0.06 radius=0.01
Joints:
- added joint base_link_back_caster_joint: type fixed, parent base_link, child back_caster, origin xyz=-0.1 0 -0.15 rpy=0 0 0
- added joint base_link_front_caster_joint: type fixed, parent base_link, child front_caster, origin xyz=0.1 0 -0.15 rpy=0 0 0
- added joint base_link_plate_joint: type fixed, parent base_footprint, child base_link, origin xyz=0 0 0.15 rpy=0 0 0
- added joint joint_base_left_wheel: type continuous, parent base_link, child link_left_wheel, origin xyz=0 -0.2 -0.15 rpy=0 0 0, axis 0 1 0, limit effort=10000 velocity=1000
- added joint joint_base_right_wheel: type continuous, parent base_link, child link_right_wheel, origin xyz=0 0.2 -0.15 rpy=0 0 0, axis 0 1 0, limit effort=10000 velocity=1000

Commit message: Add laser joint and flip it. Fix mass and inertia

File: my_rb1_description/urdf/my_rb1_robot.urdf (robot description, URDF)
Before this commit: robot rb1_robot, 6 links, 5 joints
Links:
- added link front_laser, mass 1.0
- link back_caster: mass 1 -> 0.9
- link base_link: mass 18 -> 20.2
- link front_caster: mass 1 -> 0.9
Joints:
- added joint base_link_front_laser_joint: type fixed, parent base_link, child front_laser, origin xyz=0.25 0.0 0.075 rpy=3.14159265 0 0
- joint joint_base_left_wheel: origin xyz=0 -0.2 -0.15 rpy=0 0 0 -> xyz=0 0.2 -0.15 rpy=0 0 0
- joint joint_base_right_wheel: origin xyz=0 0.2 -0.15 rpy=0 0 0 -> xyz=0 -0.2 -0.15 rpy=0 0 0

Commit message: add bridge cmd_vel, add diff-drive & LiDAR, align wheels, tweak caster height

File: my_rb1_description/urdf/my_rb1_robot.urdf (robot description, URDF)
Before this commit: robot rb1_robot, 7 links, 6 joints
Joints:
- joint base_link_back_caster_joint: origin xyz=-0.1 0 -0.15 rpy=0 0 0 -> xyz=-0.1 0 -0.1625 rpy=0 0 0
- joint base_link_front_caster_joint: origin xyz=0.1 0 -0.15 rpy=0 0 0 -> xyz=0.1 0 -0.1625 rpy=0 0 0

Commit message: save copy and replace urdf file with solution code

File: my_rb1_description/urdf/my_rb1_robot.urdf (robot description, URDF)
Before this commit: robot rb1_robot, 7 links, 6 joints
Links:
- removed link link_left_wheel
- removed link link_right_wheel
- added link left_wheel, mass 1.5; collision cylinder length=0.03 radius=0.025; visual cylinder length=0.03 radius=0.025
- added link right_wheel, mass 1.5; collision cylinder length=0.03 radius=0.025; visual cylinder length=0.03 radius=0.025
- link back_caster: mass 0.9 -> 0.5; geometry collision sphere radius=0.025; visual sphere radius=0.025
- link base_link: mass 20.2 -> 20.5; geometry collision cylinder length=0.3 radius=0.25; visual cylinder length=0.3 radius=0.25
- link front_caster: mass 0.9 -> 0.5; geometry collision sphere radius=0.025; visual sphere radius=0.025
- link front_laser: mass 1.0 -> None
Joints:
- removed joint joint_base_left_wheel
- removed joint joint_base_right_wheel
- added joint base_link_left_wheel_joint: type continuous, parent base_link, child left_wheel, origin xyz=0 0.2 -0.15 rpy=0 0 0, axis 0 1 0
- added joint base_link_right_wheel_joint: type continuous, parent base_link, child right_wheel, origin xyz=0 -0.2 -0.15 rpy=0 0 0, axis 0 1 0
- joint base_link_back_caster_joint: origin xyz=-0.1 0 -0.1625 rpy=0 0 0 -> xyz=-0.1 0.0 -0.15 rpy=0 0 0
- joint base_link_front_caster_joint: origin xyz=0.1 0 -0.1625 rpy=0 0 0 -> xyz=0.1 0.0 -0.15 rpy=0 0 0
- joint base_link_front_laser_joint: origin xyz=0.25 0.0 0.075 rpy=3.14159265 0 0 -> xyz=0.25 0 0.075 rpy=3.14 0 0

Commit message: Fix robot position

File: my_rb1_description/urdf/my_rb1_robot.urdf (robot description, URDF)
Before this commit: robot rb1_robot, 7 links, 6 joints
Joints:
- joint base_link_plate_joint: origin xyz=0 0 0.15 rpy=0 0 0 -> xyz=0 0 0.175 rpy=0 0 0
